File: Hardware/DSD_BOARD/DSD_BOARD.kicad_pcb (KiCad board)
At the start: 4 copper layers, 100 x 65 mm, 207 parts, among them J1 Conn_02x08_Odd_Even, U1 74AHC595, U10 74AHC595, U11 74AHC595, U12 74AHC595, U13 74AHC595, U14 74AHC595, U15 74AHC595, U16 74AHC595, U2 74AHC595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

Commit message: DSD Board Rev
Parts:
- added R135: 33, PCM_Resistor_SMD_AKL:R_0603_1608Metric, B.Cu at (161.8, 59.5)
- added R136: 33, PCM_Resistor_SMD_AKL:R_0603_1608Metric, B.Cu at (161.8, 62.1)
- added R137: 33, PCM_Resistor_SMD_AKL:R_0603_1608Metric, B.Cu at (161.7, 64.9)
- added R138: 33, PCM_Resistor_SMD_AKL:R_0603_1608Metric, B.Cu at (161.6, 70.0)
- added R139: 33, PCM_Resistor_SMD_AKL:R_0603_1608Metric, B.Cu at (161.6, 72.9)
- added R140: 4.7 k, PCM_Resistor_SMD_AKL:R_0603_1608Metric, B.Cu at (161.6, 67.9)
Connections:
- J1 pad 11: R_DATA_P -> Net-(J1-Pin_11)
- J1 pad 13: R_DATA_N -> Net-(J1-Pin_13)
- J1 pad 3: BCLK -> Net-(J1-Pin_3)
- J1 pad 5: L_DATA_P -> Net-(J1-Pin_5)
- J1 pad 7: L_DATA_N -> Net-(J1-Pin_7)
Routing:
- net GND: track 12.7 -> 6.56 mm, vias 47 -> 276
- net BCLK: track 279.1 -> 273.4 mm
- net R_DATA_P: track 21.9 -> 17.2 mm
- net L_DATA_N: track 20.1 -> 15.6 mm
- net L_DATA_P: track 34.5 -> 30.8 mm
- net DSD_EN: track 270.1 -> 273.4 mm
- net Net-(J1-Pin_13): track 0.00 -> 3.15 mm
- net Net-(J1-Pin_11): track 0.00 -> 3.02 mm
- net Net-(J1-Pin_3): track 0.00 -> 3.02 mm
- net Net-(J1-Pin_5): track 0.00 -> 2.96 mm
- net Net-(J1-Pin_7): track 0.00 -> 2.91 mm
- net R_DATA_N: track 33.3 -> 31.7 mm
- net +VSW: track 28.9 -> 29.4 mm, vias 32 -> 33
