File: Hardware/DSD_BOARD/DSD_BOARD.kicad_sch (KiCad schematic)
At the start: 207 parts, among them J1 Conn_02x08_Odd_Even, U1 74AHC595, U10 74AHC595, U11 74AHC595, U12 74AHC595, U13 74AHC595, U14 74AHC595, U15 74AHC595, U16 74AHC595, U2 74AHC595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

Commit message: DSD Board Rev
Parts:
- added R135, R136, R137, R138, R139: 33, PCM_Resistor_SMD_AKL:R_0603_1608Metric, symbol ERDAL:R_0603
- added R140: 4.7 k, PCM_Resistor_SMD_AKL:R_0603_1608Metric, symbol ERDAL:R_0603
Connections:
- net +VSW: now also R140.2
- net BCLK: now also R135.1; no longer J1.3 (Pin_3)
- net DSD_EN: now also R140.1
- net L_DATA_N: now also R137.1; no longer J1.7 (Pin_7)
- net L_DATA_P: now also R136.1; no longer J1.5 (Pin_5)
- net R_DATA_N: now also R139.1; no longer J1.13 (Pin_13)
- net R_DATA_P: now also R138.1; no longer J1.11 (Pin_11)
- new net: J1.7 (Pin_7), R137.2
- new net: J1.11 (Pin_11), R138.2
- new net: J1.3 (Pin_3), R135.2
- new net: J1.13 (Pin_13), R139.2
- new net: J1.5 (Pin_5), R136.2
Other:
- moved on the sheet: H1, H2, H3, H4, H5, H6, J1
