File: Hardware/MAIN_BOARD/ARTIX7.kicad_sch (KiCad schematic)
At the start: 75 parts, among them J1 Conn_01x06, J4 JTAG/SPI, SW1 SW_Push, U1 XC7A100T-CSG324, U2 W25Q128JVS, U20 TPS62130RGTT, Y2 50mhz

Commit message: some PCB/schemtic improvements
some PCB improvements,
three additional debug LEDs,
add serial res. at data/clk line
Parts:
- removed J4: JTAG/SPI, Connector_PinHeader_2.54mm:PinHeader_1x02_P2.54mm_Vertical, symbol Connector_Generic:Conn_01x02
- removed R45: 1k, Resistor_SMD:R_0603_1608Metric, symbol Erdal:R_0603
- added J15: Conn_01x04_Pin, Connector_PinHeader_2.54mm:PinHeader_1x04_P2.54mm_Vertical, symbol Connector:Conn_01x04_Pin
- added R11: 33, EP4CE_Footprint:R_0603_1608Metric, symbol Erdal:R_0603
- added R45 (x2): 22, Resistor_SMD:R_0603_1608Metric, symbol Erdal:R_0603
- added RN1, RN2, RN3: R_4x0402_Convex, PCM_Resistor_SMD_AKL:R_Array_Convex_4x0402, symbol PCM_Resistor_AKL:R_4x0402_Convex
Connections:
- net BCLK_L_F: now also RN1.3 (R3.1); no longer U1.B17 (IO_L7N_T1_AD2N_15)
- net BCLK_R_F: now also RN2.3 (R3.1); no longer U1.D18 (IO_L21N_T3_DQS_A18_15)
- net DATA_N_L_F: now also RN1.1 (R1.1); no longer U1.C17 (IO_L20N_T3_A19_15)
- net DATA_N_R_F: now also RN2.1 (R1.1); no longer U1.E18 (IO_L21P_T3_DQS_15)
- net DATA_P_L_F: now also RN1.4 (R4.1); no longer U1.A18 (IO_L10N_T1_AD11N_15)
- net DATA_P_R_F: now also RN2.4 (R4.1); no longer U1.D17 (IO_L16N_T2_A27_15)
- net DSD_A: now also RN3.3 (R3.1); no longer U1.G17 (IO_L18N_T2_A23_15)
- net DSD_A_N: now also R45.2; no longer U1.J17 (IO_L23P_T3_FOE_B_15)
- net DSD_B: now also RN3.2 (R2.1); no longer U1.G18 (IO_L22P_T3_A17_15)
- net DSD_B_N: now also R45.2; no longer U1.J18 (IO_L23N_T3_FWE_B_15)
- net DSD_CLK: now also RN3.4 (R4.1); no longer U1.F18 (IO_L22N_T3_A16_15)
- net GND: now also U1.P11 (M2_0), J15.4 (Pin_4)
- net LCLK_F: now also RN1.2 (R2.1); no longer U1.B18 (IO_L10P_T1_AD11P_15)
- net RCLK_F: now also RN2.2 (R2.1); no longer U1.E17 (IO_L16P_T2_A28_15)
- net at R11.1, Y2.3 (OUT): now also R11.1
- net I2S_IN_CLK: now reaches U1.D15 (IO_L12P_T1_MRCC_15)
- net I2S_IN_CLK: now also J15.2 (Pin_2)
- net I2S_IN_LRCLK: now reaches U1.E15 (IO_L11P_T1_SRCC_15)
- net I2S_IN_LRCLK: now also J15.1 (Pin_1)
- net I2S_IN_DATA: now reaches U1.E16 (IO_L11N_T1_SRCC_15)
- net I2S_IN_DATA: now also J15.3 (Pin_3)
- net PA11: now reaches U1.M4 (IO_L16P_T2_34)
- new net: RN1.5 (R4.2), U1.A18 (IO_L10N_T1_AD11N_15)
- new net: RN1.6 (R3.2), U1.B17 (IO_L7N_T1_AD2N_15)
- new net: RN1.7 (R2.2), U1.B18 (IO_L10P_T1_AD11P_15)
- new net: RN1.8 (R1.2), U1.C17 (IO_L20N_T3_A19_15)
- new net: RN2.5 (R4.2), U1.D17 (IO_L16N_T2_A27_15)
- new net: RN2.6 (R3.2), U1.D18 (IO_L21N_T3_DQS_A18_15)
- new net: RN2.7 (R2.2), U1.E17 (IO_L16P_T2_A28_15)
- new net: RN2.8 (R1.2), U1.E18 (IO_L21P_T3_DQS_15)
- new net: RN3.5 (R4.2), U1.F18 (IO_L22N_T3_A16_15)
- new net: RN3.6 (R3.2), U1.G17 (IO_L18N_T2_A23_15)
- new net: RN3.7 (R2.2), U1.G18 (IO_L22P_T3_A17_15)
- new net: R45.1, U1.J17 (IO_L23P_T3_FOE_B_15)
- new net: R45.1, U1.J18 (IO_L23N_T3_FWE_B_15)
- new net IO12: R11.2
- no-connect marks 84 -> 82
Other:
- moved on the sheet: R11
