File: Hardware/MAIN_BOARD/FPGA.kicad_sch (KiCad schematic)
At the start: 128 parts, among them J10 Conn_02x08_Odd_Even, J11 Conn_02x08_Odd_Even, J4 XMOS, J6 HDMI_A, J6 USB_B, U1 CS8416-xZZ, U11 SN74LVC1G04DBVR, U13 Si5342A-D, U14 USB3320C-EZK, U17 ADV7611BSWZ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

Commit message: some PCB/schemtic improvements
some PCB improvements,
three additional debug LEDs,
add serial res. at data/clk line
Parts:
- added D2 (x3): RED, LED_SMD:LED_0805_2012Metric, symbol dk_LED-Indication-Discrete:LTST-C150KRKT
- added R43 (x3): 1k, Capacitor_SMD:C_0603_1608Metric, symbol Erdal:R_0603
- added RN3: R_4x0402_Convex, PCM_Resistor_SMD_AKL:R_Array_Convex_4x0402, symbol PCM_Resistor_AKL:R_4x0402_Convex
- L7: footprint Inductor_SMD:L_1008_2520Metric -> Inductor_SMD:L_1206_3216Metric
Connections:
- net +3.3V: no longer J11.4 (Pin_4)
- net GND: now also R43.2, R43.2, R43.2
- net SPDIF_I2S_BCLK: now also RN3.3 (R3.1); no longer U1.27 (OSCLK)
- net SPDIF_I2S_DATA: now also RN3.2 (R2.1); no longer R65.2, U1.26 (SDOUT)
- net SPDIF_I2S_LRCLK: now also RN3.4 (R4.1); no longer U1.28 (OLRCK)
- new net: D2.2, R43.1 (x3)
- new net: R65.2, RN3.7 (R2.2), U1.26 (SDOUT)
- new net: RN3.5 (R4.2), U1.28 (OLRCK)
- new net: RN3.6 (R3.2), U1.27 (OSCLK)
- new net IO12: J11.4 (Pin_4)
- new net LED5: D2.1
- new net LED6: D2.1
- new net LED7: D2.1
- no-connect marks 52 -> 54
